Commit message: gazebo plugin work correctly

File: src/robot_description/a1_description/xacro/gazebo.xacro (robot description, xacro)
@@ -9,5 +9,5 @@
     </gazebo>
     <!-- Show the trajectory of trunk center. -->
-    <xacro:if value="$(arg DRAW)">
+    <xacro:if value="$(arg USE_DRAW)">
         <!-- <gazebo>
             <plugin name="3dplot" filename="libLinkPlot3DPlugin.so">

File: src/robot_description/a1_description/xacro/stereo_camera.xacro (robot description, xacro)
@@ -30,5 +30,5 @@
         <origin xyz="${d435_cam_mount_from_center_offset} ${-d435_cam_depth_py} 0" rpy="${pi/2} 0 ${pi/2}"/>
         <geometry>
-          <mesh filename="package://a1_description/meshes/realsense_d435.stl" />
+          <mesh filename="../meshes/realsense_d435.stl" />
         </geometry>
       </visual>
